File: pcb/hsync-sense/hsync-sense.kicad_pcb (KiCad board)
At the start: 2 copper layers, 23.6 x 9.5 mm, 11 parts, among them P1 CONN_01X03, U1 TSV992

Commit message: o Update resistor values.
Parts:
- D1: value PhotoDiode -> SFH203P
- R1, R2, R5: value R -> 22k
- R3, R4, R6: value R -> 2.2k
Connections:
- net +5V renamed +3V3
- net /signal-out renamed /~signal_out
