File: pcb/hsync-sense/hsync-sense.sch (KiCad schematic (older format))
At the start: 11 parts, among them P1 CONN_01X03, U1 TSV992

Commit message: o Update resistor values.
Parts:
- D1: value PhotoDiode -> SFH203P
- R1, R2, R5: value R -> 22k
- R3, R4, R6: value R -> 2.2k
Connections:
- net +5V renamed +3V3
- net signal-out renamed ~signal_out
Changed lines of the file:
@@
 LIBS:valves
 LIBS:hsync-sense-cache
-EELAYER 25 0
+EELAYER 26 0
 EELAYER END
 $Descr A4 11693 8268
@@
 P 3600 3100
 F 0 "D1" V 3554 3178 50  0000 L CNN
-F 1 "PhotoDiode" H 3400 2950 50  0000 L CNN
+F 1 "SFH203P" H 3400 2950 50  0000 L CNN
 F 2 "LEDs:LED-5MM" H 3600 3100 50  0001 C CNN
 F 3 "" H 3600 3100 50  0000 C CNN
@@
 F 3 "" H 4250 2750 50  0000 C CNN
 	1    4250 2750
-	1    0    0    -1
-$EndComp
-$Comp
-L +5V #PWR02
-U 1 1 588C0015
-P 4250 3300
-F 0 "#PWR02" H 4250 3150 50  0001 C CNN
-F 1 "+5V" H 4265 3473 50  0000 C CNN
-F 2 "" H 4250 3300 50  0000 C CNN
-F 3 "" H 4250 3300 50  0000 C CNN
-	1    4250 3300
 	1    0    0    -1
 $EndComp
@@
 Connection ~ 3850 3500
 $Comp
-L +5V #PWR04
-U 1 1 588C0320
-P 3850 2550
-F 0 "#PWR04" H 3850 2400 50  0001 C CNN
-F 1 "+5V" H 3865 2723 50  0000 C CNN
-F 2 "" H 3850 2550 50  0000 C CNN
-F 3 "" H 3850 2550 50  0000 C CNN
-	1    3850 2550
-	1    0    0    -1
-$EndComp
-$Comp
 L OP275 U1
 U 2 1 588C0351
@@
 P 4900 3550
 F 0 "R6" H 4970 3596 50  0000 L CNN
-F 1 "R" H 4970 3505 50  0000 L CNN
+F 1 "2.2k" H 4970 3505 50  0000 L CNN
 F 2 "Resistors_SMD:R_0603" V 4830 3550 50  0001 C CNN
 F 3 "" H 4900 3550 50  0000 C CNN
@@
 P 4900 2700
 F 0 "R3" H 4970 2746 50  0000 L CNN
-F 1 "R" H 4970 2655 50  0000 L CNN
+F 1 "2.2k" H 4970 2655 50  0000 L CNN
 F 2 "Resistors_SMD:R_0603" V 4830 2700 50  0001 C CNN
 F 3 "" H 4900 2700 50  0000 C CNN
@@
 Wire Wire Line
 	5600 3400 5600 3000
-$Comp
-L +5V #PWR05
-U 1 1 588C061B
-P 4900 2550
-F 0 "#PWR05" H 4900 2400 50  0001 C CNN
-F 1 "+5V" H 4915 2723 50  0000 C CNN
-F 2 "" H 4900 2550 50  0000 C CNN
-F 3 "" H 4900 2550 50  0000 C CNN
-	1    4900 2550
-	1    0    0    -1
-$EndComp
 $Comp
 L GND #PWR06
@@
 P 5250 3400
 F 0 "R5" H 5320 3446 50  0000 L CNN
-F 1 "R" H 5320 3355 50  0000 L CNN
+F 1 "22k" H 5320 3355 50  0000 L CNN
 F 2 "Resistors_SMD:R_0603" V 5180 3400 50  0001 C CNN
 F 3 "" H 5250 3400 50  0000 C CNN
@@
 P 3850 2700
 F 0 "R2" H 3700 2700 50  0000 L CNN
-F 1 "R" H 3920 2655 50  0000 L CNN
+F 1 "22k" H 3700 2550 50  0000 L CNN
 F 2 "Resistors_SMD:R_0603" V 3780 2700 50  0001 C CNN
 F 3 "" H 3850 2700 50  0000 C CNN
@@
 P 3850 3350
 F 0 "R4" H 3920 3396 50  0000 L CNN
-F 1 "R" H 3920 3305 50  0000 L CNN
+F 1 "2.2k" H 3920 3305 50  0000 L CNN
 F 2 "Resistors_SMD:R_0603" V 3780 3350 50  0001 C CNN
 F 3 "" H 3850 3350 50  0000 C CNN
@@
 P 4200 2600
 F 0 "R1" V 4150 2750 50  0000 L CNN
-F 1 "R" V 4150 2400 50  0000 L CNN
+F 1 "22k" V 4100 2400 50  0000 L CNN
 F 2 "Resistors_SMD:R_0603" V 4130 2600 50  0001 C CNN
 F 3 "" H 4200 2600 50  0000 C CNN
@@
 Wire Wire Line
 	5800 3200 5800 3250
-$Comp
-L +5V #PWR08
-U 1 1 58929AE1
-P 5800 3100
-F 0 "#PWR08" H 5800 2950 50  0001 C CNN
-F 1 "+5V" V 5850 3150 50  0000 C CNN
-F 2 "" H 5800 3100 50  0000 C CNN
-F 3 "" H 5800 3100 50  0000 C CNN
-	1    5800 3100
-	0    -1   -1   0
-$EndComp
 $Comp
 L C C2
@@
 	1    0    0    -1
 $EndComp
-$Comp
-L +5V #PWR010
-U 1 1 58929C98
-P 6000 3550
-F 0 "#PWR010" H 6000 3400 50  0001 C CNN
-F 1 "+5V" H 6015 3723 50  0000 C CNN
-F 2 "" H 6000 3550 50  0000 C CNN
-F 3 "" H 6000 3550 50  0000 C CNN
-	1    6000 3550
-	1    0    0    -1
-$EndComp
 Text Label 3650 2900 1    60   ~ 0
 PhotoIn
@@
 DivLow
 Text Label 5700 3000 1    60   ~ 0
-signal-out
+~signal_out
 $Comp
 L CONN_01X03 P1
@@
 Wire Wire Line
 	5600 3000 5800 3000
+$Comp
+L +3.3V #PWR?
+U 1 1 589E946D
+P 5800 3100
+F 0 "#PWR?" H 5800 2950 50  0001 C CNN
+F 1 "+3.3V" V 5850 3050 50  0000 L CNN
+F 2 "" H 5800 3100 50  0000 C CNN
+F 3 "" H 5800 3100 50  0000 C CNN
+	1    5800 3100
+	0    -1   -1   0
+$EndComp
+$Comp
+L +3.3V #PWR?
+U 1 1 589E9523
+P 6000 3550
+F 0 "#PWR?" H 6000 3400 50  0001 C CNN
+F 1 "+3.3V" H 6050 3650 50  0000 L CNN
+F 2 "" H 6000 3550 50  0000 C CNN
+F 3 "" H 6000 3550 50  0000 C CNN
+	1    6000 3550
+	1    0    0    -1
+$EndComp
+$Comp
+L +3.3V #PWR?
+U 1 1 589E970E
+P 4900 2550
+F 0 "#PWR?" H 4900 2400 50  0001 C CNN
+F 1 "+3.3V" H 4950 2650 50  0000 L CNN
+F 2 "" H 4900 2550 50  0000 C CNN
+F 3 "" H 4900 2550 50  0000 C CNN
+	1    4900 2550
+	1    0    0    -1
+$EndComp
+$Comp
+L +3.3V #PWR?
+U 1 1 589E973D
+P 3850 2550
+F 0 "#PWR?" H 3850 2400 50  0001 C CNN
+F 1 "+3.3V" H 3650 2700 50  0000 L CNN
+F 2 "" H 3850 2550 50  0000 C CNN
+F 3 "" H 3850 2550 50  0000 C CNN
+	1    3850 2550
+	1    0    0    -1
+$EndComp
+$Comp
+L +3.3V #PWR?
+U 1 1 589E9863
+P 4250 3300
+F 0 "#PWR?" H 4250 3150 50  0001 C CNN
+F 1 "+3.3V" H 4300 3400 50  0000 L CNN
+F 2 "" H 4250 3300 50  0000 C CNN
+F 3 "" H 4250 3300 50  0000 C CNN
+	1    4250 3300
+	1    0    0    -1
+$EndComp
 $EndSCHEMATC
