File: pcb/pocket-cape/pocket-cape.kicad_pcb (KiCad board)
At the start: 4 copper layers, 49 x 32.1 mm, 34 parts, among them J1 Sync1, J2 12V, J3 Sync2, J4 Sled, J5 Laser1, J6 PM1, J7 PM2, J8 Laser2, U1 MIC920, U2 74LVC2G14GV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

Commit message: Move component labels for better readability.
Also add signal labels on the PocketBeagle header for easier testpoint
finding.
Parts:
- J2: value 12V -> 12..16V
Other:
- board text added: "+5V"
- board text added: "GND"
- board text added: "Ls1"
- board text added: "Ls2"
- board text added: "M_CLK"
- board text added: "~EN1"
- board text added: "~EN2"
- board text added: "~S1"
- board text added: "~S2"
Changed lines of the file:
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@@
   (general
     (thickness 1.6)
-    (drawings 430)
+    (drawings 440)
     (tracks 282)
     (zones 0)
@@
   )
   (setup
-    (last_trace_width 0.5)
+    (last_trace_width 0.25)
     (user_trace_width 0.25)
     (user_trace_width 0.3)
@@
     (at 148.5011 117.7036)
     (attr virtual)
-    (fp_text reference P1 (at -22.7711 -3.6576 90) (layer F.SilkS)
+    (fp_text reference P1 (at -23.2791 -3.1496 90) (layer F.SilkS)
       (effects (font (size 1.56845 1.56845) (thickness 0.19812)))
     )
@@
     (tags "capacitor 1206")
     (attr smd)
-    (fp_text reference C4 (at 1.778 -1.778 90) (layer F.SilkS)
+    (fp_text reference C4 (at 0.132 -1.654 270) (layer F.SilkS)
       (effects (font (size 1 1) (thickness 0.15)))
     )
@@
     (tags SOD-123)
     (attr smd)
-    (fp_text reference D1 (at 1.65 -2.286 180) (layer F.SilkS)
+    (fp_text reference D1 (at -3.066 -0.59 180) (layer F.SilkS)
       (effects (font (size 1 1) (thickness 0.15)))
     )
@@
     (tags "resistor 0603")
     (attr smd)
-    (fp_text reference R6 (at -0.012 1.524 90) (layer F.SilkS)
-      (effects (font (size 1 1) (thickness 0.15)))
+    (fp_text reference R6 (at -1.536 1.27 180) (layer F.SilkS)
+      (effects (font (size 0.7 0.7) (thickness 0.15)))
     )
     (fp_text value R (at 0 1.5 90) (layer F.Fab)
@@
     (tags "resistor 0603")
     (attr smd)
-    (fp_text reference R7 (at 0 -1.524 270) (layer F.SilkS)
-      (effects (font (size 1 1) (thickness 0.15)))
+    (fp_text reference R7 (at -1.016 -1.27) (layer F.SilkS)
+      (effects (font (size 0.7 0.7) (thickness 0.15)))
     )
     (fp_text value R (at 0 1.5 270) (layer F.Fab)
@@
     (tags "TSOT-23-6 MK06A TSOT-6")
     (attr smd)
-    (fp_text reference U2 (at -3.048 0.254 180) (layer F.SilkS)
+    (fp_text reference U2 (at -2.794 1.016 180) (layer F.SilkS)
       (effects (font (size 1 1) (thickness 0.15)))
     )
@@
     (tags "inductor taiyo-yuden nr smd")
     (attr smd)
-    (fp_text reference L1 (at -2.858 -4.191) (layer F.SilkS)
+    (fp_text reference L1 (at -2.604 -4.191) (layer F.SilkS)
       (effects (font (size 1 1) (thickness 0.15)))
     )
@@
     (descr "Through hole straight pin header, 1x05, 2.54mm pitch, single row")
     (tags "Through hole pin header THT 1x05 2.54mm single row")
-    (fp_text reference J6 (at 0 -2.794 270) (layer F.SilkS)
+    (fp_text reference J6 (at 0 -2.54 270) (layer F.SilkS)
       (effects (font (size 1 1) (thickness 0.15)))
     )
@@
     (descr "Through hole straight pin header, 1x05, 2.54mm pitch, single row")
     (tags "Through hole pin header THT 1x05 2.54mm single row")
-    (fp_text reference J7 (at 0 -2.794 270) (layer F.SilkS)
+    (fp_text reference J7 (at 0 -2.54 270) (layer F.SilkS)
       (effects (font (size 1 1) (thickness 0.15)))
     )
@@
       (effects (font (size 1 1) (thickness 0.15)))
     )
-    (fp_text value Sled (at -3.81 0.508 270) (layer F.SilkS)
+    (fp_text value Sled (at 13.462 0.762 270) (layer F.SilkS)
       (effects (font (size 1 1) (thickness 0.15)))
     )
@@
     (descr "JST XH series connector, B02B-XH-A, top entry type, through hole")
     (tags "connector jst xh tht top vertical 2.50mm")
-    (fp_text reference J2 (at 1.25 -3.5 90) (layer F.SilkS)
-      (effects (font (size 1 1) (thickness 0.15)))
-    )
-    (fp_text value 12V (at 1.25 4.5 90) (layer F.Fab)
+    (fp_text reference J2 (at -0.896 1.948 90) (layer F.SilkS)
+      (effects (font (size 1 1) (thickness 0.15)))
+    )
+    (fp_text value 12..16V (at 1.39 -3.386 90) (layer F.SilkS)
       (effects (font (size 1 1) (thickness 0.15)))
     )
@@
     )
   )
+  (gr_text ~EN1 (at 129.54 89.789) (layer F.SilkS)
+    (effects (font (size 0.7 0.7) (thickness 0.15)))
+  )
+  (gr_text ~EN2 (at 132.08 89.789) (layer F.SilkS)
+    (effects (font (size 0.7 0.7) (thickness 0.15)))
+  )
+  (gr_text M_CLK (at 137.16 89.662) (layer F.SilkS)
+    (effects (font (size 0.7 0.7) (thickness 0.15)))
+  )
+  (gr_text "Ls2\n" (at 167.64 117.602) (layer F.SilkS)
+    (effects (font (size 0.8 0.8) (thickness 0.15)))
+  )
+  (gr_text Ls1 (at 149.86 117.602) (layer F.SilkS)
+    (effects (font (size 0.8 0.8) (thickness 0.15)))
+  )
+  (gr_text GND (at 144.78 117.602) (layer F.SilkS)
+    (effects (font (size 0.8 0.8) (thickness 0.15)))
+  )
+  (gr_text ~S1 (at 165.1 89.789) (layer F.SilkS)
+    (effects (font (size 0.7 0.7) (thickness 0.15)))
+  )
+  (gr_text ~S2 (at 162.56 89.789) (layer F.SilkS)
+    (effects (font (size 0.7 0.7) (thickness 0.15)))
+  )
+  (gr_text +5V (at 126.492 120.396) (layer F.SilkS)
+    (effects (font (size 0.8 0.8) (thickness 0.15)))
+  )
+  (gr_text GND (at 144.78 120.396) (layer F.SilkS)
+    (effects (font (size 0.8 0.8) (thickness 0.15)))
+  )
   (gr_text HZ (at 154.178 98.806 90) (layer F.SilkS)

Commit message: Fix wrong connection to stepper connector.
o common is not the center tap, but Pin5
o Also some more labelling (e.g. adding RX/TX)
Connections:
- J4 pad 3: VDD_5V -> Net-(J4-Pad3)
- J4 pad 5: Net-(J4-Pad5) -> VDD_5V
- J6 pad 2: Net-(J6-Pad2) -> (no net)
- J7 pad 2: Net-(J7-Pad2) -> (no net)
- P1 pad 10: /(U1.B13)SPI0.MISO -> (no net)
- P1 pad 11: /(U1.L15)USB1.D+ -> (no net)
- P1 pad 12: /(U1.B14)SPI0.MOSI -> (no net)
- P1 pad 13: /(U1.L14)USB1.ID -> (no net)
- P1 pad 14: (no net) -> Net-(P1-Pad14)
- P1 pad 17: /(U1.B9)VREF- -> (no net)
- P1 pad 18: /(U1.B7)VREF+ -> (no net)
- P1 pad 19: /(U1.A8)AIN0~1.8V -> (no net)
- P1 pad 2: /(U1.F2)AIN6~3.3V -> (no net)
- P1 pad 21: /(U1.B8)AIN1~1.8V -> (no net)
- P1 pad 23: /(U1.B6)AIN2~1.8V -> (no net)
- P1 pad 24: (no net) -> Net-(P1-Pad24)
- P1 pad 25: /(U1.C6)AIN3~1.8V -> (no net)
- P1 pad 26: /(U1.B10)I2C2.SDA -> (no net)
- P1 pad 27: /(U1.C7)AIN4~1.8V -> (no net)
- P1 pad 28: /(U1.A10)I2C2.SCL -> (no net)
- P1 pad 29: /(U1.C4)PRU-0.7 -> (no net)
- P1 pad 3: /(U1.M14)USB1.DRVVBUS -> (no net)
- P1 pad 30: /(U1.B12)UART0.TX -> (no net)
- P1 pad 31: /(U1.A3)PRU-0.4 -> (no net)
- P1 pad 32: /(U1.A12)UART0.RX -> (no net)
- P1 pad 33: /(U1.A2)PRU-0.1 -> (no net)
- P1 pad 35: /(U1.F1) -> (no net)
- P1 pad 36: /(U1.A1)PWM0A -> (no net)
- P1 pad 4: /(U1.E1) -> (no net)
- P1 pad 5: /(U1.M15)USB1.VBUS -> (no net)
- P1 pad 6: /(U1.A14)SPI0.CS -> (no net)
- P1 pad 7: USB_DC -> (no net)
- P1 pad 8: /(U1.A13)SPI0.CLK -> (no net)
- P1 pad 9: /(U1.L16)USB1.D- -> (no net)
- P2 pad 1: /(U1.P12)PWM1A -> (no net)
- P2 pad 11: /(U1.A11)I2C1.SDA -> (no net)
- P2 pad 12: /(U1.T11)PWR.BTN -> (no net)
- P2 pad 13: SYS_5V -> (no net)
- P2 pad 14: VIN.BAT -> (no net)
- P2 pad 16: /BAT.TEMP -> (no net)
- P2 pad 17: /(U1.T7) -> (no net)
- P2 pad 19: /(U1.T5) -> (no net)
- P2 pad 2: /(U1.T16) -> (no net)
- P2 pad 20: /(U1.R7) -> (no net)
- P2 pad 25: /(U1.C13)SPI1.MOSI -> (no net)
- P2 pad 26: /(U1.R11)RESET# -> (no net)
- P2 pad 27: /(U1.C12)SPI1.MISO -> (no net)
- P2 pad 28: /(U1.C3)PRU-0.6 -> (no net)
- P2 pad 29: /(U1.C5)SPI1.CLK -> (no net)
- P2 pad 3: /(U1.P5)GPIO-0.23 -> (no net)
- P2 pad 31: /(U1.A4)SPI1.CS -> (no net)
- P2 pad 34: /(U1.B3)PRU-0.5 -> (no net)
- P2 pad 35: /(U1.F3)AIN5~3.3V -> (no net)
- P2 pad 36: /(U1.N13)AIN7~1.8V -> (no net)
- P2 pad 5: /(U1.P15)UART4.RX -> (no net)
- P2 pad 7: /(U1.R16)UART4.TX -> (no net)
- P2 pad 8: /(U1.N14) -> (no net)
- P2 pad 9: /(U1.B11)I2C1.SCL -> (no net)
- U3 pad 10: (no net) -> Net-(U3-Pad10)
- U3 pad 11: (no net) -> Net-(U3-Pad11)
- U3 pad 12: (no net) -> Net-(U3-Pad12)
- U3 pad 13: Net-(J4-Pad5) -> Net-(J4-Pad4)
- U3 pad 14: Net-(J4-Pad4) -> Net-(J4-Pad3)
- U3 pad 5: (no net) -> Net-(U3-Pad5)
- U3 pad 6: (no net) -> Net-(U3-Pad6)
- U3 pad 7: (no net) -> Net-(U3-Pad7)
Routing:
- net Net-(J4-Pad5): track 5.96 -> 0.00 mm
- net Net-(J4-Pad3): track 0.00 -> 5.43 mm
- net VDD_5V: track 70.0 -> 64.9 mm
- net Net-(J4-Pad4): track 5.45 -> 4.92 mm
Other:
- board text added: "RX"
- board text added: "TX"

Commit message: Use three-way connector for Laser (GND - signal - 12V)
Parts:
- J5, J8: footprint Connectors_JST:JST_XH_B02B-XH-A_02x2.50mm_Straight -> Connectors_JST:JST_XH_B03B-XH-A_03x2.50mm_Straight
- moved J5 2.03 mm to (143.3, 111.8)
- moved J8 1.52 mm to (154.4, 111.8)
Connections:
- net STEP1 renamed STEP_A1
- net STEP2 renamed STEP_B1
- net STEP3 renamed STEP_A2
- net STEP4 renamed STEP_B2
Routing:
- net +12V: track 16.6 -> 67.3 mm
- net GND: track 161.0 -> 153.6 mm
- net LASER2: track 11.0 -> 12.6 mm
- net LASER1: track 5.48 -> 6.34 mm
- net VDD_5V: track 64.9 -> 65.6 mm
Other:
- net class Default: clearance 0 -> 0.18
- rule trace_clearance: 0 -> 0.18

Commit message: Simplyfy photo diode sync input.
o The 74LVC14 inputs are sufficiently high impedance that we
  can directly connect the photo input.
o Also: switch to JST PH 2mm connectors for laser output.
Parts:
- removed C3, C5: C, Capacitors_SMD:C_0603
- removed R1, R2, R3, R4, R8, R9: R, Resistors_SMD:R_0603
- removed REF***: OSHW-Logo2_9.8x8mm_SilkScreen, Symbols:OSHW-Logo2_9.8x8mm_SilkScreen
- removed U1, U5: MIC920, TO_SOT_Packages_SMD:SOT-23-5
- J5, J8: footprint Connectors_JST:JST_XH_B03B-XH-A_03x2.50mm_Straight -> Connectors_JST:JST_PH_B3B-PH-K_03x2.00mm_Straight
- R10, R5: value R -> 100k
- moved R10 5.98 mm to (162.1, 103.1), turned to 0 degrees
- moved J3 5.80 mm to (166.2, 106.2)
- moved J1 4.58 mm to (166.2, 99.2)
- moved C6 4.26 mm to (162.1, 101.6), turned to 0 degrees
- moved R5 2.83 mm to (162.1, 100.1), turned to 0 degrees
- moved J5 1.58 mm to (144.8, 112.0)
- moved J8 0.34 mm to (154.2, 112.0)
Connections:
- J1 pad 2: Net-(C3-Pad2) -> Net-(J1-Pad2)
- J3 pad 2: Net-(C5-Pad2) -> Net-(J3-Pad2)
- R10 pad 1: GND -> Net-(J3-Pad2)
- R10 pad 2: Net-(R10-Pad2) -> VDD_5V
- R5 pad 1: GND -> Net-(J1-Pad2)
- R5 pad 2: Net-(R2-Pad2) -> VDD_5V
- U2 pad 1: Net-(R10-Pad2) -> Net-(J3-Pad2)
- U2 pad 3: Net-(R2-Pad2) -> Net-(J1-Pad2)
Routing:
- net GND: track 153.6 -> 120.4 mm, vias 4 -> 3
- net Net-(R10-Pad2): track 15.4 -> 0.00 mm
- net Net-(J3-Pad2): track 0.00 -> 14.8 mm
- net /PhotoBias: track 14.0 -> 0.00 mm
- net Net-(C5-Pad1): track 10.1 -> 0.00 mm
- net Net-(J1-Pad2): track 0.00 -> 8.54 mm
- net VDD_5V: track 65.6 -> 57.5 mm
- net Net-(C3-Pad1): track 7.11 -> 0.00 mm
- net Net-(C3-Pad2): track 6.98 -> 0.00 mm
- net Net-(C5-Pad2): track 6.56 -> 0.00 mm
- net Net-(R2-Pad2): track 5.54 -> 0.00 mm
- net LASER2: track 12.6 -> 14.4 mm
- net LASER1: track 6.34 -> 5.65 mm
