File: pcb/pocket-cape/pocket-cape.sch (KiCad schematic (older format))
At the start: 28 parts, among them J1 Sync1, J10 Display, J11 USB1, J2 12..16V, J3 Sync2, J4 Sled, J5 Laser1, J6 PM1, J7 PM2, J8 Laser2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

Commit message: Slowly converting to current kicad.
Parts:
- C1, C2, C3, C4, C6: symbol C -> pocket-cape-rescue:C
- C5: footprint Capacitors_SMD:C_0603 -> Capacitor_SMD:C_0603_1608Metric; symbol C -> pocket-cape-rescue:C
- D1: symbol D_Schottky -> pocket-cape-rescue:D_Schottky
- J1, J2, J3: symbol CONN_01X02 -> pocket-cape-rescue:CONN_01X02
- J10: symbol CONN_01X09 -> pocket-cape-rescue:CONN_01X09
- J11, J4: symbol CONN_01X05 -> pocket-cape-rescue:CONN_01X05
- J5, J8: footprint Connectors_JST:JST_PH_B3B-PH-K_03x2.00mm_Straight -> Connector_JST:JST_PH_B3B-PH-K_1x03_P2.00mm_Vertical; symbol CONN_01X03 -> Connector_Generic:Conn_01x03
- J6, J7: footprint Pin_Headers:Pin_Header_Straight_1x05_Pitch2.54mm -> Connector_PinHeader_2.54mm:PinHeader_1x05_P2.54mm_Vertical; symbol CONN_01X05 -> Connector_Generic:Conn_01x05
- J9: symbol CONN_01X04 -> pocket-cape-rescue:CONN_01X04
- L1: symbol L -> pocket-cape-rescue:L
- P1, P2: symbol 2X18-_INCH_-0.1-TH-_35MIL-DIA_-W_O-SILK -> pocket-cape-rescue:2X18-_INCH_-0.1-TH-_35MIL-DIA_-W_O-SILK
- R10, R5, R6, R7: symbol R -> pocket-cape-rescue:R
- U1: footprint TO_SOT_Packages_SMD:SOT-23-6 -> Package_TO_SOT_SMD:SOT-23-6; symbol 74LVC2G14GV -> pocket-cape-rescue:74LVC2G14GV
- U1: footprint (none) -> Package_TO_SOT_SMD:SOT-23-6; symbol 74LVC2G14GV -> pocket-cape-rescue:74LVC2G14GV
- U3: footprint Housings_SOIC:SOIC-16_3.9x9.9mm_Pitch1.27mm -> Package_SO:SOIC-16_3.9x9.9mm_P1.27mm; symbol ULN2003A -> Transistor_Array:ULN2003A
- U4: footprint TO_SOT_Packages_SMD:SOT-23-6 -> Package_TO_SOT_SMD:SOT-23-6; symbol AP3211 -> pocket-cape-rescue:AP3211
Connections:
- net +5V: now also U3.9 (COM)
- net GND: now also U3.11 (O6), U3.14 (O3), U3.3 (I3), U3.6 (I6), U3.8 (GND); no longer U3.13 (O4), U3.15 (O2), U3.2 (I2), U3.4 (I4)
- net STEP_A1: now also U3.7 (I7); no longer U3.6 (I6)
- net STEP_A2: now also U3.2 (I2); no longer U3.1 (I1)
- net STEP_B1: now also U3.4 (I4); no longer U3.3 (I3)
- net STEP_B2: now also U3.1 (I1)
- net at U3.10 (O7): now also J4.1 (P1)
- net at J4.2 (P2): now also U3.13 (O4); no longer U3.14 (O3)
- net at J4.3 (P3): now also U3.15 (O2); no longer U3.16 (O1)
- net at J4.4 (P4): now also U3.16 (O1)
Other:
- moved on the sheet: U3
