File: pcb/pocket-cape/pocket-cape.sch (KiCad schematic (older format))
At the start: 28 parts, among them J1 Sync1, J10 Display, J11 USB1, J2 12..16V, J3 Sync2, J4 Sled, J5 Laser1, J6 PM1, J7 PM2, J8 Laser2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

Commit message: More update: convert to 5.x kicab libraries.
Parts:
- C1, C6: footprint Capacitors_SMD:C_0603 -> Capacitor_SMD:C_0603_1608Metric; symbol pocket-cape-rescue:C -> Device:C
- C2, C3, C4: footprint Capacitors_SMD:C_1206 -> Capacitor_SMD:C_1206_3216Metric; symbol pocket-cape-rescue:C -> Device:C
- C5: symbol pocket-cape-rescue:C -> Device:C
- D1: footprint Diodes_SMD:D_SOD-123 -> Diode_SMD:D_SOD-123; symbol pocket-cape-rescue:D_Schottky -> Device:D_Schottky
- J1, J3: footprint Connectors_JST:JST_PH_B2B-PH-K_02x2.00mm_Straight -> Connector_JST:JST_PH_B2B-PH-K_1x02_P2.00mm_Vertical; symbol pocket-cape-rescue:CONN_01X02 -> Connector_Generic:Conn_01x02
- J10: symbol pocket-cape-rescue:CONN_01X09 -> Connector_Generic:Conn_01x09
- J11: symbol pocket-cape-rescue:CONN_01X05 -> Connector_Generic:Conn_01x05
- J2: footprint Connectors_JST:JST_XH_B02B-XH-A_02x2.50mm_Straight -> Connector_JST:JST_XH_B2B-XH-A_1x02_P2.50mm_Vertical; symbol pocket-cape-rescue:CONN_01X02 -> Connector_Generic:Conn_01x02
- J4: footprint Connectors_JST:JST_XH_B05B-XH-A_05x2.50mm_Straight -> Connector_JST:JST_XH_B5B-XH-A_1x05_P2.50mm_Vertical; symbol pocket-cape-rescue:CONN_01X05 -> Connector_Generic:Conn_01x05
- J9: footprint Connectors_JST:JST_PH_B4B-PH-K_04x2.00mm_Straight -> Connector_JST:JST_PH_B4B-PH-K_1x04_P2.00mm_Vertical; symbol pocket-cape-rescue:CONN_01X04 -> Connector_Generic:Conn_01x04
- L1: footprint Inductors:Inductor_Taiyo-Yuden_NR-60xx -> Inductor_SMD:L_Taiyo-Yuden_NR-60xx; symbol pocket-cape-rescue:L -> Device:L
- R10, R5, R6, R7: footprint Resistors_SMD:R_0603 -> Resistor_SMD:R_0603_1608Metric; symbol pocket-cape-rescue:R -> Device:R
