File: pcb/laser-drive/laser-drive.sch (KiCad schematic (older format))
At the start: 29 parts, among them J1 CONN_01X03, P1 LaserOut, Q1 BCP5616Q, Q2 MTM232270, U2 MIC920

Commit message: o work in progress.
Parts:
- removed C5, C6, C7, C8: 10u, Capacitors_SMD:C_1210, symbol C
- C2: renamed from C9; footprint Capacitors_SMD:C_0805 -> Capacitors_SMD:C_0603
- J1: footprint Pin_Headers:Pin_Header_Straight_1x03_Pitch2.54mm -> Pin_Headers:Pin_Header_Straight_1x03_Pitch2.00mm
- P1: footprint Pin_Headers:Pin_Header_Straight_1x02 -> Connectors_JST:JST_XH_B02B-XH-A_02x2.50mm_Straight
- TP1: value Current -> Curr
- TP3: value Control-Out -> Ctrl
- renumbered C2 to C3, C3 to C4, C4 to C5, C10 to C6, C11 to C7
Other:
- moved on the sheet: C2
Changed lines of the file:
@@
-EESchema Schematic File Version 2
+EESchema Schematic File Version 3
 LIBS:power
 LIBS:laser-drive-cache
@@
 F 0 "P1" H 6877 1741 50  0000 L CNN
 F 1 "LaserOut" H 6877 1650 50  0000 L CNN
-F 2 "Pin_Headers:Pin_Header_Straight_1x02" H 6800 1700 50  0001 C CNN
+F 2 "Connectors_JST:JST_XH_B02B-XH-A_02x2.50mm_Straight" H 6800 1700 50  0001 C CNN
 F 3 "" H 6800 1700 50  0000 C CNN
 	1    6800 1700
@@
 $EndComp
 $Comp
-L C C8
-U 1 1 58D41772
-P 6550 4100
-F 0 "C8" H 6450 4200 50  0000 L CNN
-F 1 "10u" H 6500 3850 50  0000 L CNN
-F 2 "Capacitors_SMD:C_1210" H 6588 3950 50  0001 C CNN
-F 3 "" H 6550 4100 50  0000 C CNN
-	1    6550 4100
-	1    0    0    -1
-$EndComp
-$Comp
-L C C9
+L C C2
 U 1 1 58D41773
-P 6800 4100
-F 0 "C9" H 6700 4200 50  0000 L CNN
-F 1 "100n" H 6750 3850 50  0000 L CNN
-F 2 "Capacitors_SMD:C_0805" H 6838 3950 50  0001 C CNN
-F 3 "" H 6800 4100 50  0000 C CNN
-	1    6800 4100
+P 6000 4100
+F 0 "C2" H 5900 4200 50  0000 L CNN
+F 1 "100n" H 5950 3850 50  0000 L CNN
+F 2 "Capacitors_SMD:C_0603" H 6038 3950 50  0001 C CNN
+F 3 "" H 6000 4100 50  0000 C CNN
+	1    6000 4100
 	1    0    0    -1
 $EndComp
@@
 $EndComp
 $Comp
-L C C7
-U 1 1 58D41783
-P 6350 4100
-F 0 "C7" H 6250 4200 50  0000 L CNN
-F 1 "10u" H 6300 3850 50  0000 L CNN
-F 2 "Capacitors_SMD:C_1210" H 6388 3950 50  0001 C CNN
-F 3 "" H 6350 4100 50  0000 C CNN
-	1    6350 4100
-	1    0    0    -1
-$EndComp
-$Comp
-L C C6
-U 1 1 58D41784
-P 6150 4100
-F 0 "C6" H 6050 4200 50  0000 L CNN
-F 1 "10u" H 6100 3850 50  0000 L CNN
-F 2 "Capacitors_SMD:C_1210" H 6188 3950 50  0001 C CNN
-F 3 "" H 6150 4100 50  0000 C CNN
-	1    6150 4100
-	1    0    0    -1
-$EndComp
-$Comp
 L C C5
-U 1 1 58D41785
-P 5950 4100
-F 0 "C5" H 5850 4200 50  0000 L CNN
-F 1 "10u" H 5900 3850 50  0000 L CNN
-F 2 "Capacitors_SMD:C_1210" H 5988 3950 50  0001 C CNN
-F 3 "" H 5950 4100 50  0000 C CNN
-	1    5950 4100
-	1    0    0    -1
-$EndComp
-$Comp
-L C C4
 U 1 1 58D41786
 P 5750 4100
-F 0 "C4" H 5650 4200 50  0000 L CNN
+F 0 "C5" H 5650 4200 50  0000 L CNN
 F 1 "10u" H 5700 3850 50  0000 L CNN
 F 2 "Capacitors_SMD:C_1210" H 5788 3950 50  0001 C CNN
@@
 $EndComp
 $Comp
-L C C3
+L C C4
 U 1 1 58D41787
 P 5550 4100
-F 0 "C3" H 5450 4200 50  0000 L CNN
+F 0 "C4" H 5450 4200 50  0000 L CNN
 F 1 "10u" H 5400 4000 50  0000 L CNN
 F 2 "Capacitors_SMD:C_1210" H 5588 3950 50  0001 C CNN
@@
 $EndComp
 $Comp
-L C C2
+L C C3
 U 1 1 58D41788
 P 5350 4100
-F 0 "C2" H 5250 4200 50  0000 L CNN
+F 0 "C3" H 5250 4200 50  0000 L CNN
 F 1 "10u" H 5200 4000 50  0000 L CNN
 F 2 "Capacitors_SMD:C_1210" H 5388 3950 50  0001 C CNN
@@
 P 6000 1650
 F 0 "TP1" V 6200 1850 50  0000 C CNN
-F 1 "Current" V 6100 1850 50  0000 C CNN
+F 1 "Curr" V 6100 1850 50  0000 C CNN
 F 2 "Measurement_Points:Measurement_Point_Round-SMD-Pad_Small" H 6103 1724 50  0001 C CNN
 F 3 "" H 6200 1650 50  0000 C CNN
@@
 P 5450 2000
 F 0 "TP3" H 5450 2250 50  0000 C CNN
-F 1 "Control-Out" H 5450 2200 50  0000 C CNN
+F 1 "Ctrl" H 5450 2200 50  0000 C CNN
 F 2 "Measurement_Points:Measurement_Point_Round-SMD-Pad_Small" H 5553 2074 50  0001 C CNN
 F 3 "" H 5650 2000 50  0000 C CNN
@@
 	5750 3900 5750 3950
 Connection ~ 5750 3900
-Wire Wire Line
-	5950 3900 5950 3950
-Connection ~ 5950 3900
-Wire Wire Line
-	6150 3900 6150 3950
-Connection ~ 6150 3900
-Wire Wire Line
-	6350 3900 6350 3950
-Connection ~ 6350 3900
-Wire Wire Line
-	6550 3900 6550 3950
-Connection ~ 6550 3900
-Connection ~ 6550 4250
-Connection ~ 6350 4250
-Connection ~ 6150 4250
-Connection ~ 5950 4250
 Connection ~ 5750 4250
 Connection ~ 5550 4250
@@
 Connection ~ 5050 1250
 Wire Wire Line
-	5350 4250 6800 4250
-Wire Wire Line
-	6800 3900 6800 3950
-Wire Wire Line
-	5350 3900 6800 3900
+	6000 3900 6000 3950
 Connection ~ 5450 2000
 Wire Wire Line
@@
 ControlOut
 $Comp
-L C C11
+L C C7
 U 1 1 58D86FB5
 P 5200 1400
-F 0 "C11" V 5350 1300 50  0000 L CNN
+F 0 "C7" V 5350 1300 50  0000 L CNN
 F 1 "100n" V 5150 1500 50  0000 L CNN
 F 2 "Capacitors_SMD:C_0603" H 5238 1250 50  0001 C CNN
@@
 F 0 "J1" H 4969 2925 50  0000 C CNN
 F 1 "CONN_01X03" V 5150 3250 50  0000 C CNN
-F 2 "Pin_Headers:Pin_Header_Straight_1x03_Pitch2.54mm" H 5050 3250 50  0001 C CNN
+F 2 "Pin_Headers:Pin_Header_Straight_1x03_Pitch2.00mm" H 5050 3250 50  0001 C CNN
 F 3 "" H 5050 3250 50  0001 C CNN
 	1    5050 3250
@@
 $EndComp
 $Comp
-L C C10
+L C C6
 U 1 1 59B52DAB
 P 5600 2200
-F 0 "C10" V 5750 2050 50  0000 L CNN
+F 0 "C6" V 5750 2050 50  0000 L CNN
 F 1 "100p" V 5750 2250 50  0000 L CNN
 F 2 "Capacitors_SMD:C_0603" H 5638 2050 50  0001 C CNN
@@
 	5750 2200 5750 2000
 Connection ~ 5750 2000
+Wire Wire Line
+	5350 3900 6000 3900
+Wire Wire Line
+	5350 4250 6000 4250
 $EndSCHEMATC
